File: kicad/water.tank/water.tank.sch (KiCad schematic (older format))
At the start: 7 parts, among them J1 ESP8266, J5 5V, U1 LD33V

Commit message: a few unrelated things
Parts:
- 5V1: renamed from J5; value 5V -> source
- OLED1: value OLED -> OLED1
- SENSOR1: value SENSOR -> JSN
Connections:
- net CH_PC renamed CH_PD
Changed lines of the file:
@@
 ADC
 Text GLabel 3850 2650 0    50   Input ~ 0
-CH_PC
+CH_PD
 Text GLabel 3850 2750 0    50   Input ~ 0
 IO16
@@
 P 4850 3800
 F 0 "OLED1" H 4650 4000 50  0000 L CNN
-F 1 "OLED" H 4650 4050 50  0001 L CNN
+F 1 "OLED1" H 4650 4050 50  0001 L CNN
 F 2 "Connector_JST:JST_EH_B4B-EH-A_1x04_P2.50mm_Vertical" H 4850 3800 50  0001 C CNN
 F 3 "~" H 4850 3800 50  0001 C CNN
@@
 $EndComp
 $Comp
-L Connector:Conn_01x02_Female J5
+L Connector:Conn_01x02_Female 5V1
 U 1 1 62840F2A
 P 7150 2550
-F 0 "J5" H 7178 2526 50  0000 L CNN
-F 1 "5V" H 7178 2435 50  0000 L CNN
+F 0 "5V1" H 7178 2526 50  0000 L CNN
+F 1 "source" H 7178 2435 50  0001 L CNN
 F 2 "Connector_JST:JST_EH_B2B-EH-A_1x02_P2.50mm_Vertical" H 7150 2550 50  0001 C CNN
 F 3 "~" H 7150 2550 50  0001 C CNN
@@
 P 4450 3700
 F 0 "SENSOR1" H 4200 3400 50  0000 L CNN
-F 1 "SENSOR" H 4342 3367 50  0001 C CNN
+F 1 "JSN" H 4342 3367 50  0001 C CNN
 F 2 "Connector_PinSocket_2.54mm:PinSocket_1x04_P2.54mm_Vertical" H 4450 3700 50  0001 C CNN
 F 3 "~" H 4450 3700 50  0001 C CNN
